File: Hardware/Depth Sensor/depth-sensor/depth-sensor.kicad_sch (KiCad schematic)
At the start: 33 parts, among them J1 Conn_01x02_Female, J2 Conn_01x04_Female, J3 Conn_01x04_Female, Q1 Q_NMOS_GSD, Q2 Q_PMOS_GSD, U1 LM358, U2 LM358, U3 TL431DBZ

Commit message: Depth-Sensor: Routing and PCB layout
Also update .gitignore to KiCAD 6
Parts:
- added H1, H2, H3, H4: MountingHole, MountingHole:MountingHole_3.2mm_M3, symbol Mechanical:MountingHole
- C1, C10, C2, C3, C4, C5, C6, C7, C8, C9: footprint (none) -> Capacitor_SMD:C_0402_1005Metric
- J1: footprint (none) -> Connector_PinHeader_2.54mm:PinHeader_1x02_P2.54mm_Vertical
- J2, J3: footprint (none) -> Connector_PinHeader_2.54mm:PinHeader_1x04_P2.54mm_Vertical
- Q1, Q2: footprint (none) -> Package_TO_SOT_SMD:SOT-23
- R1, R11, R12, R13, R14, R17, R18, R2, R3, R4, R5, R7, R8: footprint (none) -> Resistor_SMD:R_0402_1005Metric
- RV1: footprint (none) -> Potentiometer_THT:Potentiometer_Vishay_T73YP_Vertical; LCSC PN (none) -> C118956
- RV2: renamed from RV?; value 200 -> 500; footprint (none) -> Potentiometer_THT:Potentiometer_Vishay_T73YP_Vertical; LCSC PN (none) -> C118916
- U1, U2: footprint (none) -> Package_SO:SOP-8_3.9x4.9mm_P1.27mm
