File: Hardware/Depth Sensor/depth-sensor.kicad_sch (KiCad schematic)
At the start: 37 parts, among them J1 Conn_01x02_Female, J2 Conn_01x04_Female, J3 Conn_01x04_Female, Q1 Q_NMOS_GSD, Q2 Q_PMOS_GSD, U1 LM358, U2 LM358, U3 TL431DBZ

Commit message: Depth Sensor: CAM
Also fixed folder structure
Parts:
- added R?: ~, Resistor_SMD:R_0402_1005Metric, symbol Device:R_Small
Connections:
- net VDD: now also R?.2
- net at C5.2, C7.2, RV1.2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: now also R?.1
Other:
- note added: "DNP"
Changed lines of the file:
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@@
   (junction (at 125.73 109.22) (diameter 0) (color 0 0 0 0)
   )
+  (junction (at 116.84 96.52) (diameter 0) (color 0 0 0 0)
+  )
   (junction (at 62.23 113.03) (diameter 0) (color 0 0 0 0)
   )
@@
   (junction (at 118.11 64.77) (diameter 0) (color 0 0 0 0)
   )
+  (junction (at 124.46 102.87) (diameter 0) (color 0 0 0 0)
+  )
   (junction (at 153.67 121.92) (diameter 0) (color 0 0 0 0)
   )
@@
     (stroke (width 0) (type default) (color 0 0 0 0))
   )
+  (wire (pts (xy 124.46 97.79) (xy 124.46 96.52))
+    (stroke (width 0) (type default) (color 0 0 0 0))
+  )
+  (wire (pts (xy 124.46 96.52) (xy 116.84 96.52))
+    (stroke (width 0) (type default) (color 0 0 0 0))
+  )
   (wire (pts (xy 187.96 130.81) (xy 187.96 128.27))
     (stroke (width 0) (type default) (color 0 0 0 0))
@@
     (stroke (width 0) (type default) (color 0 0 0 0))
   )
+  (wire (pts (xy 124.46 102.87) (xy 129.54 102.87))
+    (stroke (width 0) (type default) (color 0 0 0 0))
+  )
   (wire (pts (xy 78.74 125.73) (xy 78.74 127))
     (stroke (width 0) (type default) (color 0 0 0 0))
   )
-  (wire (pts (xy 121.92 102.87) (xy 129.54 102.87))
+  (wire (pts (xy 121.92 102.87) (xy 124.46 102.87))
     (stroke (width 0) (type default) (color 0 0 0 0))
   )
@@
   (wire (pts (xy 68.58 69.85) (xy 74.93 69.85))
     (stroke (width 0) (type default) (color 0 0 0 0))
+  )
+  (text "DNP" (at 123.19 101.6 90)
+    (effects (font (size 1.27 1.27)) (justify left bottom))
   )
   (text "GAIN" (at 101.6 71.12 0)
@@
     (pin "8")
   )
+  (symbol (lib_id "Device:R_Small") (at 124.46 100.33 180) (unit 1)
+    (in_bom yes) (on_board yes)
+    (property "Reference" "R?" (id 0) (at 124.46 95.25 0))
+    (property "Value" "~" (id 1) (at 124.46 95.25 0))
+    (property "Footprint" "Resistor_SMD:R_0402_1005Metric" (id 2) (at 124.46 100.33 0)
+      (effects (font (size 1.27 1.27)) hide)
+    )
+    (property "Datasheet" "~" (id 3) (at 124.46 100.33 0)
+      (effects (font (size 1.27 1.27)) hide)
+    )
+    (pin "1")
+    (pin "2")
+  )
   (symbol (lib_id "Device:R_Small") (at 69.85 111.76 180) (unit 1)
     (in_bom yes) (on_board yes)
@@
       (reference "R18") (unit 1) (value "330") (footprint "Resistor_SMD:R_0402_1005Metric")
     )
+    (path "/860c370c-8ce3-45b3-854f-48797382da6c"
+      (reference "R?") (unit 1) (value "~") (footprint "Resistor_SMD:R_0402_1005Metric")
+    )
     (path "/41c8e294-2b28-4d75-b1ec-e326133a3d04"

Commit message: Project: remove obsolete copies from directory
Parts:
- gave numbers to parts that had none: 1
Changed lines of the file:
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@@
   (symbol (lib_id "Device:R_Small") (at 171.45 77.47 90) (unit 1)
     (in_bom yes) (on_board yes)
-    (property "Reference" "R18" (id 0) (at 171.45 74.93 90))
+    (property "Reference" "R18" (id 0) (at 171.45 81.28 90))
     (property "Value" "330" (id 1) (at 171.45 79.398 90))
     (property "Footprint" "Resistor_SMD:R_0402_1005Metric" (id 2) (at 171.45 77.47 0)
@@
   (symbol (lib_id "Device:R_Small") (at 124.46 100.33 180) (unit 1)
     (in_bom yes) (on_board yes)
-    (property "Reference" "R?" (id 0) (at 124.46 95.25 0))
+    (property "Reference" "R6" (id 0) (at 124.46 95.25 0))
     (property "Value" "~" (id 1) (at 124.46 95.25 0))
     (property "Footprint" "Resistor_SMD:R_0402_1005Metric" (id 2) (at 124.46 100.33 0)
@@
   (symbol (lib_id "Device:R_Small") (at 163.83 82.55 0) (unit 1)
     (in_bom yes) (on_board yes)
-    (property "Reference" "R17" (id 0) (at 166.37 82.55 90))
-    (property "Value" "330" (id 1) (at 161.902 82.55 90))
+    (property "Reference" "R17" (id 0) (at 160.02 83.82 0))
+    (property "Value" "330" (id 1) (at 160.02 81.28 0))
     (property "Footprint" "Resistor_SMD:R_0402_1005Metric" (id 2) (at 163.83 82.55 0)
       (effects (font (size 1.27 1.27)) hide)
@@
       (reference "R5") (unit 1) (value "100") (footprint "Resistor_SMD:R_0402_1005Metric")
     )
+    (path "/860c370c-8ce3-45b3-854f-48797382da6c"
+      (reference "R6") (unit 1) (value "~") (footprint "Resistor_SMD:R_0402_1005Metric")
+    )
     (path "/4a250130-af4d-4ae2-823a-e5173c28bea0"
       (reference "R7") (unit 1) (value "10k") (footprint "Resistor_SMD:R_0402_1005Metric")
@@
       (reference "R18") (unit 1) (value "330") (footprint "Resistor_SMD:R_0402_1005Metric")
     )
-    (path "/860c370c-8ce3-45b3-854f-48797382da6c"
-      (reference "R?") (unit 1) (value "~") (footprint "Resistor_SMD:R_0402_1005Metric")
-    )
     (path "/41c8e294-2b28-4d75-b1ec-e326133a3d04"
